File: hardware/calculator/calculator.kicad_sch (KiCad schematic)
At the start: 25 parts, among them J1 Waveshare 2.0 LCD, SW1 Matrix Key, SW10 Matrix Key, SW11 Matrix Key, SW12 Matrix Key, SW13 Matrix Key, SW14 Matrix Key, SW15 Matrix Key, SW16 Matrix Key, SW17 Power Switch, SW2 Matrix Key, SW3 Matrix Key, SW4 Matrix Key, SW5 Matrix Key, SW6 Matrix Key, SW7 Matrix Key, SW8 Matrix Key, SW9 Matrix Key, U1 XIAO-ESP32-C3-SMD, U2 PCF8574T

Commit message: v1.1: minor bug fixes
Parts:
- removed C1: 100nF, symbol Device:C
- removed U2: PCF8574T, Package_SO:SOIC-16W_7.5x10.3mm_P1.27mm, symbol Interface_Expansion:PCF8574T
- added C1: 100nF, symbol Device:C_Small
- added D1, D10, D11, D12, D13, D14, D15, D16, D17, D18, D19, D2, D20, D3, D4, D5, D6, D7, D8, D9: 1N4148W, Diode_SMD:D_SOD-123, symbol Diode:1N4148W
- added SW18, SW19, SW20, SW21: Matrix Key, symbol Switch:SW_Push
- added U2: MCP23017, Package_DIP:DIP-28_W7.62mm, symbol Interface_Expansion:MCP23017x-x-SP
- U1: value XIAO-ESP32-C3-SMD -> XIAO-ESP32-C3
- renumbered BT1 to BT, J1 to J, SW17 to SW
Connections:
- net 3V3: now also C1.1, U2.18 (~{RESET}), U2.9 (V_{DD})
- net COL1: now also SW18.2, U2.1 (GPB0)
- net COL2: now also SW19.2, U2.2 (GPB1)
- net COL3: now also SW20.2, U2.3 (GPB2)
- net COL4: now also SW21.2, U2.4 (GPB3)
- net GND: now also C1.2, U2.10 (V_{SS}), U2.15 (A0), U2.16 (A1), U2.17 (A2)
- net KBD_INT: now also U2.20 (INTA)
- net ROW1: now also D1.2 (A), D2.2 (A), D3.2 (A), D4.2 (A), U2.21 (GPA0); no longer SW1.1, SW2.1, SW3.1, SW4.1
- net ROW2: now also D5.2 (A), D6.2 (A), D7.2 (A), D8.2 (A), U2.22 (GPA1); no longer SW5.1, SW6.1, SW7.1, SW8.1
- net ROW3: now also D10.2 (A), D11.2 (A), D12.2 (A), D9.2 (A), U2.23 (GPA2); no longer SW10.1, SW11.1, SW12.1, SW9.1
- net ROW4: now also D13.2 (A), D14.2 (A), D15.2 (A), D16.2 (A), U2.24 (GPA3); no longer SW13.1, SW14.1, SW15.1, SW16.1
- net SCL: now also U2.12 (SCK)
- net SDA: now also U2.13 (SDA)
- new net: D19.1 (K), SW20.1
- new net: D7.1 (K), SW7.1
- new net: D2.1 (K), SW2.1
- new net: D14.1 (K), SW14.1
- new net: D3.1 (K), SW3.1
- new net: D20.1 (K), SW21.1
- new net: D8.1 (K), SW8.1
- new net: D11.1 (K), SW11.1
- new net: D6.1 (K), SW6.1
- new net: D17.1 (K), SW18.1
- new net: D12.1 (K), SW12.1
- new net: D16.1 (K), SW16.1
- new net: D1.1 (K), SW1.1
- new net: D5.1 (K), SW5.1
- new net: D15.1 (K), SW15.1
- new net: D4.1 (K), SW4.1
- new net: D18.1 (K), SW19.1
- new net: D13.1 (K), SW13.1
- new net: D9.1 (K), SW9.1
- new net: D10.1 (K), SW10.1
- new net ROW5: D17.2 (A), D18.2 (A), D19.2 (A), D20.2 (A), U2.25 (GPA4)
- no-connect marks 10 -> 18
Other:
- moved on the sheet: J, R1, R2, R3

Commit message: v1.2: Minor Fixes
Parts:
- removed C1: 100nF, symbol Device:C_Small
- removed R1, R2: 4.7k, symbol Device:R
- removed R3: 10kΩ, symbol Device:R
- removed U1: XIAO-ESP32-C3, Seeed_Studio_XIAO_Series:XIAO-ESP32-C3-SMD, symbol Seeed_Studio_XIAO_Series:XIAO-ESP32-C3-SMD
- removed U2: MCP23017, Package_DIP:DIP-28_W7.62mm, symbol Interface_Expansion:MCP23017x-x-SP
- added U: Waveshare RP2040 Plus, Module:RaspberryPi_Pico_Common_Unspecified, symbol MCU_Module:RaspberryPi_Pico
Connections:
- net COL1: now also U.15 (GPIO11)
- net COL2: now also U.16 (GPIO12)
- net COL3: now also U.17 (GPIO13)
- net COL4: now also U.19 (GPIO14)
- net GND: now also U.13 (GND), U.18 (GND), U.23 (GND), U.28 (GND), U.3 (GND), U.33 (AGND), U.38 (GND), U.8 (GND)
- net MOSI: now also U.25 (GPIO19)
- net ROW1: now also U.9 (GPIO6)
- net ROW2: now also U.10 (GPIO7)
- net ROW3: now also U.11 (GPIO8)
- net ROW4: now also U.12 (GPIO9)
- net ROW5: now also U.14 (GPIO10)
- net SCK: now also U.24 (GPIO18)
- net TFT_BL: now also U.27 (GPIO21)
- net TFT_CS: now also U.22 (GPIO17)
- net TFT_DC: now also U.21 (GPIO16)
- net TFT_RST: now also U.26 (GPIO20)
- net VBAT: now reaches SW.1 (A)
- net VBAT: now also U.39 (VSYS)
- net 3V3 renamed +3V3
- net +3V3: now also U.36 (3V3)
- no-connect marks 18 -> 16
Other:
- note added: "2026-07-18"
- note added: "Calculator v2"
- note added: "Components: Waveshare RP2040 Plus / 3.7V 550mAh Li-Po Battery / Waveshare 2.0 LCD / 5*4 key matrix"
- note added: "v2: Components updated. Wiring added."
- note removed: "12-07-26"
- note removed: "Calculator v1"
- note removed: "v1: Initial schematic. Changes may apply."
- moved on the sheet: BT, J, SW
